File: lab6/Exercise 1/Exercise 1.kicad_sch (KiCad schematic)
At the start: 6 parts, among them J1 9V, SW1 SW_SPDT

Commit message: lab 6 complete
Parts:
- C1: footprint (none) -> Capacitor_THT:C_Radial_D5.0mm_H5.0mm_P2.00mm
- D1: footprint (none) -> LED_THT:LED_D5.0mm
- J1: footprint (none) -> Connector_JST:JST_PH_B2B-PH-K_1x02_P2.00mm_Vertical
- R1: footprint (none) -> Resistor_THT:R_Axial_DIN0516_L15.5mm_D5.0mm_P20.32mm_Horizontal
- R2: footprint (none) -> Resistor_THT:R_Axial_DIN0516_L15.5mm_D5.0mm_P20.32mm_Horizontal; Spice_Model (none) -> 2.2k; Spice_Netlist_Enabled (none) -> Y; Spice_Primitive (none) -> R
- SW1: footprint (none) -> Button_Switch_THT:SW_E-Switch_EG1224_SPDT_Angled
Changed lines of the file:
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@@
       (effects (font (size 1.27 1.27)) (justify right))
     )
-    (property "Footprint" "" (id 2) (at 168.91 87.63 0)
+    (property "Footprint" "LED_THT:LED_D5.0mm" (id 2) (at 168.91 87.63 0)
       (effects (font (size 1.27 1.27)) hide)
     )
@@
       (effects (font (size 1.27 1.27)) (justify left))
     )
-    (property "Footprint" "" (id 2) (at 147.0152 87.63 0)
+    (property "Footprint" "Capacitor_THT:C_Radial_D5.0mm_H5.0mm_P2.00mm" (id 2) (at 147.0152 87.63 0)
       (effects (font (size 1.27 1.27)) hide)
     )
@@
       (effects (font (size 1.27 1.27)) (justify left))
     )
-    (property "Footprint" "" (id 2) (at 167.132 77.47 90)
+    (property "Footprint" "Resistor_THT:R_Axial_DIN0516_L15.5mm_D5.0mm_P20.32mm_Horizontal" (id 2) (at 167.132 77.47 90)
       (effects (font (size 1.27 1.27)) hide)
     )
@@
     (property "Reference" "SW1" (id 0) (at 137.16 68.58 0))
     (property "Value" "SW_SPDT" (id 1) (at 137.16 71.12 0))
-    (property "Footprint" "" (id 2) (at 137.16 76.2 0)
+    (property "Footprint" "Button_Switch_THT:SW_E-Switch_EG1224_SPDT_Angled" (id 2) (at 137.16 76.2 0)
       (effects (font (size 1.27 1.27)) hide)
     )
@@
     (property "Reference" "R2" (id 0) (at 123.19 71.12 90))
     (property "Value" "2.2k" (id 1) (at 123.19 73.66 90))
-    (property "Footprint" "" (id 2) (at 123.19 79.248 90)
+    (property "Footprint" "Resistor_THT:R_Axial_DIN0516_L15.5mm_D5.0mm_P20.32mm_Horizontal" (id 2) (at 123.19 79.248 90)
       (effects (font (size 1.27 1.27)) hide)
     )
     (property "Datasheet" "~" (id 3) (at 123.19 77.47 0)
+      (effects (font (size 1.27 1.27)) hide)
+    )
+    (property "Spice_Primitive" "R" (id 4) (at 123.19 77.47 0)
+      (effects (font (size 1.27 1.27)) hide)
+    )
+    (property "Spice_Model" "2.2k" (id 5) (at 123.19 77.47 0)
+      (effects (font (size 1.27 1.27)) hide)
+    )
+    (property "Spice_Netlist_Enabled" "Y" (id 6) (at 123.19 77.47 0)
       (effects (font (size 1.27 1.27)) hide)
     )
@@
     (property "Reference" "J1" (id 0) (at 108.585 76.2 0))
     (property "Value" "9V" (id 1) (at 108.585 78.74 0))
-    (property "Footprint" "" (id 2) (at 107.95 81.28 0)
+    (property "Footprint" "Connector_JST:JST_PH_B2B-PH-K_1x02_P2.00mm_Vertical" (id 2) (at 107.95 81.28 0)
       (effects (font (size 1.27 1.27)) hide)
     )
@@
   (symbol_instances
     (path "/151e97cf-c28b-4297-94e1-1f4e40720f2e"
-      (reference "C1") (unit 1) (value "4.7uF") (footprint "")
+      (reference "C1") (unit 1) (value "4.7uF") (footprint "Capacitor_THT:C_Radial_D5.0mm_H5.0mm_P2.00mm")
     )
     (path "/0767d662-2d08-41cb-8aa6-cf96c7157767"
-      (reference "D1") (unit 1) (value "LED") (footprint "")
+      (reference "D1") (unit 1) (value "LED") (footprint "LED_THT:LED_D5.0mm")
     )
     (path "/e73e9f5d-73b9-441e-b2de-c2a838f2277f"
-      (reference "J1") (unit 1) (value "9V") (footprint "")
+      (reference "J1") (unit 1) (value "9V") (footprint "Connector_JST:JST_PH_B2B-PH-K_1x02_P2.00mm_Vertical")
     )
     (path "/2e2373fa-6616-4162-a622-03abd3a7bd6f"
-      (reference "R1") (unit 1) (value "20k") (footprint "")
+      (reference "R1") (unit 1) (value "20k") (footprint "Resistor_THT:R_Axial_DIN0516_L15.5mm_D5.0mm_P20.32mm_Horizontal")
     )
     (path "/976ed87d-fb14-4a04-8b5f-35adb83334c9"
-      (reference "R2") (unit 1) (value "2.2k") (footprint "")
+      (reference "R2") (unit 1) (value "2.2k") (footprint "Resistor_THT:R_Axial_DIN0516_L15.5mm_D5.0mm_P20.32mm_Horizontal")
     )
     (path "/57f199a6-caf0-4f4f-9898-c0915a01508e"
-      (reference "SW1") (unit 1) (value "SW_SPDT") (footprint "")
+      (reference "SW1") (unit 1) (value "SW_SPDT") (footprint "Button_Switch_THT:SW_E-Switch_EG1224_SPDT_Angled")
     )
   )
